File: ibm5161-backplane.kicad_sch (KiCad schematic)
At the start: 33 parts, among them J1 Bus_ISA_8bit, J2 Bus_ISA_8bit, J3 Bus_ISA_8bit, J4 Bus_ISA_8bit, J5 Bus_ISA_8bit, J6 Bus_ISA_8bit, J7 Bus_ISA_8bit, J8 Bus_ISA_8bit, P1 Conn_01x06, P2 Conn_01x06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

Commit message: Fixed break in +5V trace near pin B29 of slot 1. Moved finalized files to folder gerber_to_order
Parts:
- P1, P2: value Conn_01x06 -> Molex 15-48-0106
Changed lines of the file:
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@@
       (effects (font (size 1.27 1.27)) (justify left))
     )
-    (property "Value" "Conn_01x06" (at 91.44 158.75 0)
+    (property "Value" "Molex 15-48-0106" (at 91.44 158.75 0)
       (effects (font (size 1.27 1.27)) (justify left) hide)
     )
@@
       (effects (font (size 1.27 1.27)) (justify left))
     )
-    (property "Value" "Conn_01x06" (at 101.6 125.73 0)
+    (property "Value" "Molex 15-48-0106" (at 101.6 125.73 0)
       (effects (font (size 1.27 1.27)) (justify left) hide)
     )
